File: CM4-Beaglebone/CM4-Beaglebone.kicad_sch (KiCad schematic)
At the start: 29 parts, among them J1 Conn_01x03, J2 Conn_02x07_Odd_Even, J3 Conn_01x03, J7 Micro_SD_Card_Det, J9 THD-02-R, P8 BeagleBone_Black_Header, P9 BeagleBone_Black_Header, U1 TPD4EUSB30, U18 RT9742GGJ5, U2 TPD4EUSB30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

Commit message: Update Schematic
Connections:
- net nPWR_LED: no longer U5.2
- net SCL0 renamed I2C-SCL
- net SDA0 renamed I2C-SDA
Other:
- note added: "License CERN-OHL-P https://ohwr.org/cern_ohl_p_v2.txt"
- company: © 2020-2022 Raspberry Pi Ltd (formerly Raspberry Pi (Trading) Ltd.) -> (none)
- title: Compute Module 4 IO Board - GPIO - Ethernet -> BeagleBone CM4 - GPIO - Ethernet
- moved on the sheet: D1, R10, TP5, U5
